File: hardware/out/silentband.kicad_sch (KiCad schematic)
At the start: 107 parts, among them J1 Electrodes, J2 IMU, J3 USB-C, J4 LiPo 1S, Q1 AO3401A, Q2 AO3401A, SW1 RESET, SW2 BOOT, SW3 POWER, U1 ADS1298IPAGR, U2 ADS1298IPAGR, U3 ESP32-S3-WROOM-1-N8, U4 USBLC6-2SC6, U5 MCP73831T-2ACI/OT, U6 AP2112K-3.3TRG1, U7 LP5907MFX-3.0/NOPB

Commit message: Apply Fable review: slave reset timing, tantalum VCAP1, clocks on F.Cu, low-battery stop
Co-Authored-By: Claude <noreply@anthropic.com>
Parts:
- C20, C32: footprint Capacitor_SMD:C_0603_1608Metric -> Capacitor_Tantalum_SMD:CP_EIA-3216-18_Kemet-A; symbol Device:C_Small -> Device:C_Polarized_Small; LCSC C59461 -> C7183
Other:
- moved on the sheet: C21, C22, C23, C24, C25, C26, C27, C28, C29, C30, C31, C33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
