File: hardware/out/utter.kicad_sch (KiCad schematic)
At the start: 107 parts, among them J1 Electrodes, J2 IMU, J3 USB-C, J4 LiPo 1S, Q1 AO3401A, Q2 AO3401A, SW1 RESET, SW2 BOOT, SW3 POWER, U1 ADS1298IPAGR, U2 ADS1298IPAGR, U3 ESP32-S3-WROOM-1-N8, U4 USBLC6-2SC6, U5 MCP73831T-2ACI/OT, U6 AP2112K-3.3TRG1, U7 LP5907MFX-3.0/NOPB

Commit message: Rename the product to Utter (formerly SilentBand / SilentTyping)
The board, Mac app, utter CLI and Python package, firmware, mDNS (utter.local), docs and landing page all use the new name.
The board was regenerated with build.sh --reuse-route (new flag). The copper is identical to the reviewed layout, DRC/ERC are clean, and the BOM and CPL are unchanged.
USAGE paths point to the renamed repo folder (utter/).
Other:
- title: SilentBand v1 -> Utter v1
